File: Phase_2/Catch_the_light_Phase_2 Rev A_first_submit/Schematic.brd (EAGLE design)
At the start: 60 x 94 mm, 43 parts, among them U1 ATMEGA328PB-AUR

Commit message: Most current version of the board
Parts:
- added C6: 100n, rcl:C0805
- added Q2: SI2323DS, SI2323DS:SOT23
- added R18: 10k, rcl:R0805
- added R19, R20: 0, rcl:R0805
- added S2: DTSM-6, switch-tact:DTSM-6
- added U$1, U$2, U$3, U$4, U$5: TEST_POINT, My-library_:TEST_POINT
- added U$6: PINHEADER, My-library_:HEADERPIN
- added U$7, U$8, U$9: FIDUCIAL, adafruit:FIDUCIAL_1MM
- C1, C2, C3, C4, C5: value (none) -> 100n
- LED1: value (none) -> Green
- LED10, LED11, LED12, LED13, LED14, LED15, LED3, LED4, LED6, LED7, LED8, LED9: value (none) -> Red
- LED16, LED2: value (none) -> Blue
- R1, R10, R11, R12, R13, R14, R15, R16, R2, R3, R4, R5, R6, R7, R8, R9: value (none) -> 1.5k
- R17: value (none) -> 10k
- moved C2 12.8 mm to (21.8, 40.1)
- moved BATT 11.9 mm to (30.0, 65.0)
- moved C3 5.00 mm to (13.7, 40.1), turned to 0 degrees
- moved Q1 2.16 mm to (17.8, 36.2)
Connections:
- net N$3 renamed LED12
- removed net N$12: LED1.A, U1.1
- removed net N$16: ISP1.4, LED10.A, TC1.4, U1.15
- removed net N$6: LED5.A, U1.28
- new net LED1: LED1.A, U$1.P$1, U1.1
- new net LED13: LED13.A, U$4.P$1, U1.12
- new net LED5: LED5.A, U$2.P$1, U1.28
- new net PB5: ISP1.3, TC1.3, U1.17
- new net PC0: R19.1, R20.2, U1.23
- new net PC1: C6.1, R18.1, S2.1, S2.2, U1.24
- new net PD4: U$6.1, U1.2
- new net PE0: U$6.2, U1.3
- new net PE1: U$6.3, U1.6
- new net PE2: U$6.4, U1.19
- net +3V3: now also Q2.2, R18.2, R19.2, U$5.P$1; no longer BATT.1, BATT.2
- net GND: now also C6.2, Q2.1, R20.1, S2.3, S2.4
- net N$2: now also BATT.1, BATT.2, Q2.3; no longer LED13.A, U1.12
- net PB3: now also ISP1.4, LED10.A, TC1.4, U1.15; no longer ISP1.3, TC1.3, U1.17
- net PB4: now also U$3.P$1
Routing:
- net N$16: track 129.0 -> 0.00 mm, vias 1 -> 0
- net PB3: track 41.1 -> 127.6 mm, vias 2 -> 1
- net LED5: track 0.00 -> 54.0 mm
- net LED13: track 0.00 -> 53.8 mm
- net N$6: track 52.9 -> 0.00 mm
- net PB5: track 0.00 -> 41.1 mm, vias 0 -> 2
- net GND: track 37.9 -> 0.00 mm
- net PC1: track 0.00 -> 37.4 mm
- net PE2: track 0.00 -> 31.5 mm, vias 0 -> 1
- net PE1: track 0.00 -> 29.5 mm, vias 0 -> 1
- net PE0: track 0.00 -> 25.4 mm, vias 0 -> 1
- net PD4: track 0.00 -> 23.4 mm, vias 0 -> 1
- net N$2: track 52.2 -> 37.0 mm
- net PB4: track 136.1 -> 121.5 mm
- net PC0: track 0.00 -> 14.1 mm
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Other:
- outline, holes or cut-outs redrawn
