File: Phase_2/Catch_the_light_Phase_2 Rev A_first_submit/Schematic.sch (EAGLE design)
At the start: 43 parts, among them U1 ATMEGA328PB-AUR

Commit message: Most current version of the board
Parts:
- added C6: 100n, rcl:C-USC0805
- added Q2: SI2323DS, SI2323DS:SI2323DS
- added R18: 10k, rcl:R-EU_R0805
- added R19, R20: 0, rcl:R-EU_R0805
- added S2: DTSM-6, switch-tact:DTSM-6
- added U$1, U$2, U$3, U$4, U$5: TEST_POINT, My-library_:TEST_POINT
- added U$6: PINHEADER, My-library_:PINHEADER
- added U$7, U$8, U$9: FIDUCIAL, adafruit:FIDUCIAL
- C1, C2, C3, C4, C5: value (none) -> 100n
- LED1: value (none) -> Green
- LED10, LED11, LED12, LED13, LED14, LED15, LED3, LED4, LED6, LED7, LED8, LED9: value (none) -> Red
- LED16, LED2: value (none) -> Blue
- R1, R10, R11, R12, R13, R14, R15, R16, R2, R3, R4, R5, R6, R7, R8, R9: value (none) -> 1.5k
- R17: value (none) -> 10k
Connections:
- net N$17 renamed PB5
- net N$3 renamed LED12
- removed net N$12: LED1.A, U1.PD3
- removed net N$6: LED5.A, U1.PC5
- new net LED1: LED1.A, U$1.TP, U1.PD3
- new net LED13: LED13.A, U$4.TP, U1.PB0
- new net LED5: LED5.A, U$2.TP, U1.PC5
- new net PC0: R19.1, R20.2, U1.PC0
- new net PC1: C6.1, R18.1, S2.1, S2.2, U1.PC1
- new net PD4: U$6.1, U1.PD4
- new net PE0: U$6.2, U1.PE0
- new net PE1: U$6.3, U1.PE1
- new net PE2: U$6.4, U1.PE2
- net +3V3: now also Q2.S, R18.2, R19.2, U$5.TP; no longer BATT.+V@1, BATT.+V@2
- net GND: now also C6.2, Q2.G, R20.1, S2.3, S2.4
- net N$2: now also BATT.+V@1, BATT.+V@2, Q2.D; no longer LED13.A, U1.PB0
- net PB4: now also U$3.TP
Other:
- note added: "PB there incease qtouch does not work"
- note added: "Pull up and Pull Down circuit To be used for switching between qtouch and PB"
- note added: "These are test point amoung the board that will allow physical debuging"
- moved on the sheet: C1, C2, C3, C4, C5, ISP1, Q1, TC1
