File: Phase_2/Catch_the_light_Phase_2 Rev A/Schematic.sch (EAGLE design)
At the start: 58 parts, among them Q2 SI2323DS, U1 ATMEGA328PB-AUR

Commit message: Most current version of the board
Parts:
- added U$10: UMASSLGOARNIE, My-library_:UMASSLGOARNIE
- added U$11: ECE_LOGO, My-library_:ECE_LOGO
- added U$12: UMDLOGO, My-library_:UMDLOGO
Other:
- note added: "1"
- note added: "Battery/Board protection from reversed battery"
- note added: "Decoupling caps"
- note added: "For production programming"
- note added: "PB there incase qtouch does not work"
- note added: "SPI connector to be used for debugging"
- note added: "These are test point amoung the board that will allow physical debugging"
- note added: "Unused pins Atmega328pb"
- note removed: "PB there incease qtouch does not work"
- note removed: "These are test point amoung the board that will allow physical debuging"

Commit message: Add files via upload
Parts:
- LED5: value (none) -> RED
- renumbered BATT to CR2032
Changed lines of the file:
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@@
 <part name="GND3" library="supply1" library_urn="urn:adsk.eagle:library:371" deviceset="GND" device=""/>
 <part name="GND4" library="supply1" library_urn="urn:adsk.eagle:library:371" deviceset="GND" device=""/>
-<part name="BATT" library="My-library_" deviceset="BC-2003" device="SMD"/>
+<part name="CR2032" library="My-library_" deviceset="BC-2003" device="SMD"/>
 <part name="C1" library="rcl" library_urn="urn:adsk.eagle:library:334" deviceset="C-US" device="C0805" package3d_urn="urn:adsk.eagle:package:23617/2" value="100n"/>
 <part name="GND2" library="supply1" library_urn="urn:adsk.eagle:library:371" deviceset="GND" device=""/>
@@
 <part name="R6" library="rcl" library_urn="urn:adsk.eagle:library:334" deviceset="R-EU_" device="R0805" package3d_urn="urn:adsk.eagle:package:23553/2" value="1.5k"/>
 <part name="R5" library="rcl" library_urn="urn:adsk.eagle:library:334" deviceset="R-EU_" device="R0805" package3d_urn="urn:adsk.eagle:package:23553/2" value="1.5k"/>
-<part name="LED5" library="led" library_urn="urn:adsk.eagle:library:259" deviceset="LED" device="CHIP-LED0805" package3d_urn="urn:adsk.eagle:package:15818/2"/>
+<part name="LED5" library="led" library_urn="urn:adsk.eagle:library:259" deviceset="LED" device="CHIP-LED0805" package3d_urn="urn:adsk.eagle:package:15818/2" value="RED"/>
 <part name="LED4" library="led" library_urn="urn:adsk.eagle:library:259" deviceset="LED" device="CHIP-LED0805" package3d_urn="urn:adsk.eagle:package:15818/2" value="Red"/>
 <part name="R4" library="rcl" library_urn="urn:adsk.eagle:library:334" deviceset="R-EU_" device="R0805" package3d_urn="urn:adsk.eagle:package:23553/2" value="1.5k"/>
@@
 <attribute name="VALUE" x="27.94" y="139.7" size="1.778" layer="96"/>
 </instance>
-<instance part="BATT" gate="G$1" x="177.8" y="109.22" smashed="yes"/>
+<instance part="CR2032" gate="G$1" x="177.8" y="109.22" smashed="yes"/>
 <instance part="C1" gate="G$1" x="200.66" y="137.16" smashed="yes" rot="R90">
 <attribute name="NAME" x="200.025" y="138.176" size="1.778" layer="95" rot="R90"/>
@@
 <attribute name="VALUE" x="307.34" y="162.56" size="1.778" layer="96" rot="R180"/>
 </instance>
-<instance part="U$6" gate="G$1" x="111.76" y="30.48" smashed="yes">
-<attribute name="NAME" x="116.84" y="35.56" size="2.54" layer="95" rot="R90"/>
-</instance>
+<instance part="U$6" gate="G$1" x="111.76" y="30.48" smashed="yes"/>
 <instance part="Q2" gate="G$1" x="195.58" y="129.54" smashed="yes" rot="R180">
 <attribute name="VALUE" x="193.03616875" y="132.08383125" size="1.78068125" layer="96" rot="R180"/>
@@
 </segment>
 <segment>
-<pinref part="BATT" gate="G$1" pin="GND"/>
+<pinref part="CR2032" gate="G$1" pin="GND"/>
 <pinref part="GND2" gate="1" pin="GND"/>
 <wire x1="162.306" y1="110.616" x2="157.48" y2="110.616" width="0.1524" layer="91"/>
@@
 <segment>
 <wire x1="195.58" y1="115.076" x2="195.58" y2="105.616" width="0.1524" layer="91"/>
-<pinref part="BATT" gate="G$1" pin="+V@2"/>
+<pinref part="CR2032" gate="G$1" pin="+V@2"/>
 <wire x1="187.226" y1="105.616" x2="195.58" y2="105.616" width="0.1524" layer="91"/>
-<pinref part="BATT" gate="G$1" pin="+V@1"/>
+<pinref part="CR2032" gate="G$1" pin="+V@1"/>
 <wire x1="187.226" y1="115.076" x2="195.58" y2="115.076" width="0.1524" layer="91"/>
 <pinref part="Q2" gate="G$1" pin="D"/>
